Commit message: ekf

File: hyperlync_simulator_2/hyperlync_robot/robot_description/urdf/andbot.xacro (robot description, xacro)
@@ -50,4 +50,30 @@
 	<origin xyz="0.07 0 ${radius_wheel+0.135}" rpy="0 0 0"/>
   </joint>
+<joint name="IMU_joint" type="fixed">
+    <axis xyz="1 0 0"/>
+        <origin xyz="0.0 0.0 0.04"/>
+	    <parent link="base_link"/>
+	    <child link="IMU_link"/>
+</joint>
+<link name="IMU_link">
+  <inertial>
+      <mass value="0.001"/>
+          <origin rpy="0 0 0" xyz="0 0 0"/>
+	      <inertia ixx="0.0001" ixy="0" ixz="0" iyy="0.000001" iyz="0" izz="0.0001"/>
+  </inertial>
+  <visual>
+	<origin rpy="0 0 0" xyz="0 0 0"/>
+          <geometry>
+	       <box size="0.01 0.01 0.01"/>
+	  </geometry>
+        <material name="red"/>
+	  </visual>
+	    <collision>
+	    <origin rpy="0 0 0" xyz="0 0 0"/>
+		 <geometry>
+	          <box size=".01 .01 .01"/>
+		 </geometry>
+	    </collision>
+</link>
 <!-- Base link -->
   <link name="base_link">
